Commit message: fix to issue #3 , Using outdated xacro file for motoman sia20d arm

File: godel_robot_config/urdf/sia20d_workspace.urdf (robot description, URDF)
Before this commit: robot sia20d_workspace, 24 links, 23 joints
Links:
- removed link tcp
- added link tool0
- link base_link: geometry collision mesh filename=package://motoman_sia20d_support/meshes/sia20d/collision/MO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; visual mesh filename=package://motoman_sia20d_support/meshes/sia20d/visual/MOTOM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
- link link_b: geometry collision mesh filename=package://motoman_sia20d_support/meshes/sia20d/collision/MO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; visual mesh filename=package://motoman_sia20d_support/meshes/sia20d/visual/MOTOM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
- link link_e: geometry collision mesh filename=package://motoman_sia20d_support/meshes/sia20d/collision/MO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; visual mesh filename=package://motoman_sia20d_support/meshes/sia20d/visual/MOTOM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
- link link_l: geometry collision mesh filename=package://motoman_sia20d_support/meshes/sia20d/collision/MO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; visual mesh filename=package://motoman_sia20d_support/meshes/sia20d/visual/MOTOM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
- link link_r: geometry collision mesh filename=package://motoman_sia20d_support/meshes/sia20d/collision/MO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; visual mesh filename=package://motoman_sia20d_support/meshes/sia20d/visual/MOTOM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
- link link_s: geometry collision mesh filename=package://motoman_sia20d_support/meshes/sia20d/collision/MO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; visual mesh filename=package://motoman_sia20d_support/meshes/sia20d/visual/MOTOM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
- link link_t: geometry collision mesh filename=package://motoman_sia20d_support/meshes/sia20d/collision/MO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; visual mesh filename=package://motoman_sia20d_support/meshes/sia20d/visual/MOTOM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
- link link_u: geometry collision mesh filename=package://motoman_sia20d_support/meshes/sia20d/collision/MO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; visual mesh filename=package://motoman_sia20d_support/meshes/sia20d/visual/MOTOM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
Joints:
- removed joint wrist_to_tcp
- added joint link_t-tool0: type fixed, parent link_t, child tool0, origin xyz=0 0 0.0 rpy=0 0 -3.1416

File: godel_robot_config/urdf/sia20d_workspace.xacro (robot description, xacro)
@@ -1,5 +1,5 @@
 <?xml version="1.0" ?>
 <robot name="sia20d_workspace" xmlns:xacro="http://ros.org/wiki/xacro">
-	<xacro:include filename="$(find motoman_config)/cfg/sia20d_mesh_macro.xacro"/>
+	<xacro:include filename="$(find motoman_sia20d_support)/urdf/sia20d_macro.xacro"/>
 	<xacro:include filename="$(find godel_robot_config)/urdf/workspace_components.xacro"/>
 	<xacro:include filename="$(find godel_robot_config)/urdf/kinect_sensor_macro.xacro"/>
@@ -26,5 +26,5 @@
 	<!-- end of sensor definitions -->
 	<!-- instantiating arm  -->
-	<xacro:sia20d_mesh prefix="${arm_prefix}"/>
+	<xacro:motoman_sia20d prefix="${arm_prefix}"/>
 	<!-- start of arm-workcell joint definitions -->
 	<joint name="world_to_base" type="fixed">
@@ -39,11 +39,3 @@
 	</joint>
 	<!-- end of arm-workcell joint definitions -->
-	<!-- start of wrist to tcp coupling -->
-	<link name="${arm_prefix}tcp"/>
-	<joint name="${arm_prefix}wrist_to_tcp" type="fixed">
-		<parent link="${arm_prefix}link_t"/>
-		<child link="${arm_prefix}tcp"/>
-		<origin xyz="0 0 0" rpy="0 0 0"/>
-	</joint>
-	<!-- end of wrist to tcp coupling -->
 </robot>

Commit message: regenerated urdf file to reflect changes in originating xacro files

File: godel_robot_config/urdf/sia20d_workspace.urdf (robot description, URDF)
Before this commit: robot sia20d_workspace, 34 links, 33 joints
Joints:
- joint asus_mount_to_asus_link: origin xyz=0 0 0 rpy=0.0 0.0 0.0 -> xyz=0 0 0 rpy=3.14 0.0 0.0
- joint world_to_roof1: origin xyz=0.987 0 1.20 rpy=0 0 0 -> xyz=0.987 0 1.40 rpy=0 0 0

Commit message: increased length of collision model for the workcell roof

File: godel_robot_config/urdf/sia20d_workspace.urdf (robot description, URDF)
Before this commit: robot sia20d_workspace, 34 links, 33 joints
Links:
- link roof1: geometry collision box size=1.40 2.220 0.04
Joints:
- joint world_to_roof1: origin xyz=0.987 0 1.40 rpy=0 0 0 -> xyz=0.65 0 1.32 rpy=0 0 0

File: godel_robot_config/urdf/sia20d_workspace.xacro (robot description, xacro)
@@ -18,5 +18,5 @@
 		<collision>
 			<geometry>
-				<box size="1.010 2.220 0.04"/>
+				<box size="1.40 2.220 0.04"/>
 			</geometry>
 		</collision>
@@ -43,5 +43,5 @@
 		<parent link="world_frame"/>
 		<child link="roof1"/>
-		<origin xyz="0.987 0 1.40" rpy="0 0 0"/>
+		<origin xyz="0.65 0 1.32" rpy="0 0 0"/>
 	</joint>
 	<!-- end of arm-workcell joint definitions -->
