Commit message: added calibration data to camera models in the xacro files

File: godel_robot_config/urdf/asus_sensor_macro.xacro (robot description, xacro)
@@ -55,5 +55,5 @@
 			<parent link="${prefix}asus_frame"/>
 			<child link="${prefix}asus_ir_link"/>
-			<origin rpy="0 0 0" xyz="0 0 0"/>
+			<origin rpy="0 0 0" xyz="0 0.0476 0"/>
 		</joint>
 		<joint name="${prefix}asus_ir_optical_frame_joint" type="fixed">
@@ -65,5 +65,5 @@
 			<parent link="${prefix}asus_ir_link"/>
 			<child link="${prefix}asus_rgb_link"/>
-			<origin rpy="0 0 0" xyz="0 -0.03 0"/>
+			<origin rpy="0 0 0" xyz="0 -0.025 0"/>
 		</joint>
 		<joint name="${prefix}asus_rgb_optical_frame_joint" type="fixed">

File: godel_robot_config/urdf/blending_eff_macro.xacro (robot description, xacro)
@@ -30,5 +30,5 @@
 			<link name="${prefix}asus_mount"/>
 		<xacro:asus_sensor_definitions prefix="${prefix}" parent_link="${prefix}asus_mount"
-				x_val="0" y_val="-0.08" z_val="0.02" roll="3.14" pitch="0.05" yaw="0.0"/>
+				x_val="0.01479" y_val="0.006741" z_val="0.007162" roll="-3.123031" pitch="0.001618" yaw="0.02739"/>
 		<!-- joint definitions -->
 			<joint name="${prefix}gripper_to_palm" type="fixed">
