Commit message: added ATI end effector to URDF

File: godel_robot_config/urdf/sia20d_workspace.xacro (robot description, xacro)
@@ -3,8 +3,9 @@
 	<xacro:include filename="$(find motoman_sia20d_support)/urdf/sia20d_macro.xacro"/>
 	<xacro:include filename="$(find godel_robot_config)/urdf/workspace_components.xacro"/>
+	<xacro:include filename="$(find godel_robot_config)/urdf/blending_eff_macro.xacro"/>
 	<xacro:include filename="$(find godel_robot_config)/urdf/kinect_sensor_macro.xacro"/>
 	<!-- property list -->
 	<xacro:property name="workcell_height" value="1"/>
-	<xacro:property name="coupler_height" value="0.087"/>
+	<xacro:property name="coupler_height" value="0.0"/> <!--"0.087"-->
         <xacro:property name="attached_object_length" value="0.10"/>
 	<xacro:property name="attached_object_width" value="0.10"/>
@@ -26,5 +27,11 @@
 	<!-- end of sensor definitions -->
 	<!-- instantiating arm  -->
+	<xacro:blending_eff_definition eff_adjustment="0.0"/>
 	<xacro:motoman_sia20d prefix="${arm_prefix}"/>
+	<joint name="link_t_to_eff" type="fixed">
+		<parent link="link_t"/>
+		<child link="eff_frame"/>
+		<origin xyz="0 ${coupler_height} 0" rpy="0.0 0.0 0.0"/>
+	</joint>
 	<!-- start of arm-workcell joint definitions -->
 	<joint name="world_to_base" type="fixed">

Commit message: moved roof to a slightly higher position

File: godel_robot_config/urdf/sia20d_workspace.xacro (robot description, xacro)
@@ -43,5 +43,5 @@
 		<parent link="world_frame"/>
 		<child link="roof1"/>
-		<origin xyz="0.987 0 1.20" rpy="0 0 0"/>
+		<origin xyz="0.987 0 1.40" rpy="0 0 0"/>
 	</joint>
 	<!-- end of arm-workcell joint definitions -->

Commit message: made eef_frame a child link of tool0 in the robot

File: godel_robot_config/urdf/sia20d_workspace.xacro (robot description, xacro)
@@ -30,7 +30,7 @@
 	<xacro:motoman_sia20d prefix="${arm_prefix}"/>
 	<joint name="link_t_to_eff" type="fixed">
-		<parent link="link_t"/>
+		<parent link="tool0"/>
 		<child link="eff_frame"/>
-		<origin xyz="0 ${coupler_height} 0" rpy="0.0 0.0 0.0"/>
+		<origin xyz="0 ${coupler_height} 0" rpy="0.0 0.0 3.1416"/>
 	</joint>
 	<!-- start of arm-workcell joint definitions -->
