Commit message: added abb robot workspace and moveit config to godel blending

File: godel_robot_config/urdf/irb6640_workspace.xacro (robot description, xacro)
@@ -1,11 +1,11 @@
 <?xml version="1.0" ?>
-<robot name="sia20d_workspace" xmlns:xacro="http://ros.org/wiki/xacro">
-	<xacro:include filename="$(find motoman_sia20d_support)/urdf/sia20d_macro.xacro"/>
-	<xacro:include filename="$(find godel_robot_config)/urdf/workspace_components_swri.xacro"/>
+<robot name="irb6640_workspace" xmlns:xacro="http://ros.org/wiki/xacro">
+	<xacro:include filename="$(find abb_irb6600_support)/urdf/irb6640_macro.xacro"/>
+	<xacro:include filename="$(find godel_robot_config)/urdf/workspace_components.xacro"/>
 	<xacro:include filename="$(find godel_robot_config)/urdf/blending_eff_macro.xacro"/>
 	<!-- property list -->
 	<xacro:property name="workcell_height" value="1"/>
 	<xacro:property name="coupler_height" value="0.0"/> <!--"0.087"-->
-    <xacro:property name="attached_object_length" value="0.10"/>
+  <xacro:property name="attached_object_length" value="0.10"/>
 	<xacro:property name="attached_object_width" value="0.10"/>
 	<xacro:property name="attached_object_height" value="0.025"/>
@@ -13,5 +13,5 @@
 	<xacro:property name="no_go_height" value="0.1"/>
 	<!-- instantiating workcell definitions -->
-	<xacro:workcell_swri_zone1_components/>
+	<xacro:workcell_zone1_components/>
 	<!-- end of workcell definitions -->
 	<link name="roof1">
@@ -21,5 +21,5 @@
 			</geometry>
 		</collision>
-	</link>-
+	</link>
 	<link name="no_go_zone">
 		<collision>
@@ -31,5 +31,5 @@
 	<!-- instantiating arm  -->
 	<xacro:blending_eff_definition prefix="${arm_prefix}" eff_adjustment="0.0575"/>
-	<xacro:motoman_sia20d prefix="${arm_prefix}"/>
+	<xacro:abb_irb6640 prefix="${arm_prefix}"/>
 	<joint name="link_t_to_eff" type="fixed">
 		<parent link="tool0"/>

File: godel_robot_config/urdf/workspace_components_swri.xacro (robot description, xacro)
@@ -1,4 +1,4 @@
 <?xml version="1.0" ?>
-<robot name="workspace_components" xmlns:xacro="http://ros.org/wiki/xacro">
+<robot name="mantis_workspace_components" xmlns:xacro="http://ros.org/wiki/xacro">
 	<!-- property list -->
 	<xacro:property name="workcell_height" value="1"/>
@@ -62,5 +62,5 @@
 	<link name="world_frame"/>
 	<!-- workcell part1 components macro -->
-	<xacro:macro name="workcell_zone1_components">
+	<xacro:macro name="workcell_swri_zone1_components">
 		<link name="table_base1">
 			<visual>
@@ -84,5 +84,5 @@
 			<origin xyz="${workcell_length * 0.25} 0 0" rpy="0 0 0"/>
 		</joint>
-		<!-- <xacro:workcell_element name="front_wall1" parent="world_frame"
+		<xacro:workcell_element name="front_wall1" parent="world_frame"
 			 length="0.1" width="2.220" height="${workcell_height}" offset_x="1.3375" offset_y="0"/>
 		<xacro:workcell_element name="back_wall1" parent="world_frame"
@@ -93,9 +93,9 @@
 			 length="1.221" width="0.1" height="${workcell_height}" offset_x="0.687" offset_y="-1.060"/>
 		<xacro:workcell_element name="pole1" parent="world_frame"
-			length="0.09" width="0.09" height="${workcell_height}" offset_x="0.9465" offset_y="-0.845"/> -->
+			length="0.09" width="0.09" height="${workcell_height}" offset_x="0.9465" offset_y="-0.845"/>
 	</xacro:macro>
 	<!-- end of workcell part1 components macro -->
 	<!-- workcell part2 components macro -->
-	<xacro:macro name="workcell_zone2_components">
+	<!-- <xacro:macro name="workcell_zone2_components">
 		<link name="table_base2">
 			<visual>
@@ -145,5 +145,5 @@
 		<xacro:workcell_element name="cover_part2" parent="world_frame"
 			 length="0.121" width="0.260" height="0.14" offset_x="-0.012" offset_y="-0.465"/>
-	</xacro:macro>
+	</xacro:macro> -->
 	<!-- end of workcell part2 components macro -->
 </robot>
