Commit message: Cleaned up the URDFs a bit

File: godel_robot_config/urdf/irb2400_workspace.xacro (robot description, xacro)
@@ -7,29 +7,13 @@
   <xacro:property name="workcell_height" value="1"/>
   <xacro:property name="coupler_height" value="0.0"/> <!--"0.087"-->
-  <xacro:property name="attached_object_length" value="0.10"/>
-  <xacro:property name="attached_object_width" value="0.10"/>
-  <xacro:property name="attached_object_height" value="0.025"/>
   <xacro:property name="arm_prefix" value=""/>
   <xacro:property name="no_go_height" value="0.1"/>
   <!-- instantiating workcell definitions -->
   <xacro:workcell_zone1_components/>
-  <!-- end of workcell definitions -->
-<!--   <link name="roof1">
-    <collision>
-      <geometry>
-        <box size="1.40 2.220 0.04"/>
-      </geometry>
-    </collision>
-  </link> -->
-  <link name="no_go_zone">
-    <collision>
-      <geometry>
-        <box size="0.8 2.220 ${no_go_height}"/>
-      </geometry>
-    </collision>
-  </link>
   <!-- instantiating arm  -->
+  <xacro:abb_irb2400 prefix="${arm_prefix}"/>
+  <!-- instantiating end effector  -->
   <xacro:blending_eff_definition prefix="${arm_prefix}" eff_adjustment="0.0575"/>
-  <xacro:abb_irb2400 prefix="${arm_prefix}"/>
+  <!-- Attach the end effector to the end of the robot arm (tool0) -->
   <joint name="link_t_to_eff" type="fixed">
     <parent link="tool0"/>
@@ -43,9 +27,14 @@
     <origin xyz="0.241 0 0" rpy="0 0 0"/>
   </joint>
-<!--   <joint name="world_to_roof1" type="fixed">
-    <parent link="world_frame"/>
-    <child link="roof1"/>
-    <origin xyz="0.65 0 1.32" rpy="0 0 0"/>
-  </joint> -->
+  <!-- As a work-around for the lack of collision detection with move-it joint
+     moves with the work objects, we use a no-go-zone to prevent the robot
+     from getting too close to the table. Descartes is still unawares, though -->
+  <link name="no_go_zone">
+    <collision>
+      <geometry>
+        <box size="0.8 2.220 ${no_go_height}"/>
+      </geometry>
+    </collision>
+  </link>
   <joint name="world_to_no_go" type="fixed">
     <parent link="world_frame" />
@@ -53,4 +42,3 @@
     <origin xyz="1.0 0 ${no_go_height/2.0} " />
   </joint>
-  <!-- end of arm-workcell joint definitions -->
 </robot>

File: godel_robot_config/urdf/irb6640_workspace.xacro (robot description, xacro)
@@ -1,56 +1,44 @@
 <?xml version="1.0" ?>
 <robot name="irb6640_workspace" xmlns:xacro="http://ros.org/wiki/xacro">
-	<xacro:include filename="$(find abb_irb6600_support)/urdf/irb6640_macro.xacro"/>
-	<xacro:include filename="$(find godel_robot_config)/urdf/workspace_components.xacro"/>
-	<xacro:include filename="$(find godel_robot_config)/urdf/blending_eff_macro.xacro"/>
-	<!-- property list -->
-	<xacro:property name="workcell_height" value="1"/>
-	<xacro:property name="coupler_height" value="0.0"/> <!--"0.087"-->
-  <xacro:property name="attached_object_length" value="0.10"/>
-	<xacro:property name="attached_object_width" value="0.10"/>
-	<xacro:property name="attached_object_height" value="0.025"/>
-	<xacro:property name="arm_prefix" value=""/>
-	<xacro:property name="no_go_height" value="0.1"/>
-	<!-- instantiating workcell definitions -->
-	<xacro:workcell_zone1_components/>
-	<!-- end of workcell definitions -->
-	<link name="roof1">
-		<collision>
-			<geometry>
-				<box size="1.40 2.220 0.04"/>
-			</geometry>
-		</collision>
-	</link>
-	<link name="no_go_zone">
-		<collision>
-			<geometry>
-				<box size="0.8 2.220 ${no_go_height}"/>
-			</geometry>
-		</collision>
-	</link>
-	<!-- instantiating arm  -->
-	<xacro:blending_eff_definition prefix="${arm_prefix}" eff_adjustment="0.0575"/>
-	<xacro:abb_irb6640 prefix="${arm_prefix}"/>
-	<joint name="link_t_to_eff" type="fixed">
-		<parent link="tool0"/>
-		<child link="eff_frame"/>
-		<origin xyz="0 ${coupler_height} 0" rpy="0.0 0.0 3.1416"/>
-	</joint>
-	<!-- start of arm-workcell joint definitions -->
-	<joint name="world_to_base" type="fixed">
-		<parent link="world_frame"/>
-		<child link="${arm_prefix}base_link"/>
-		<origin xyz="0.241 0 0" rpy="0 0 0"/>
-	</joint>
-	<joint name="world_to_roof1" type="fixed">
-		<parent link="world_frame"/>
-		<child link="roof1"/>
-		<origin xyz="0.65 0 1.32" rpy="0 0 0"/>
-	</joint>
-	<joint name="world_to_no_go" type="fixed">
-		<parent link="world_frame" />
-		<child link="no_go_zone" />
-		<origin xyz="1.0 0 ${no_go_height/2.0} " />
-	</joint>
-	<!-- end of arm-workcell joint definitions -->
+  <xacro:include filename="$(find abb_irb6600_support)/urdf/irb6640_macro.xacro"/>
+  <xacro:include filename="$(find godel_robot_config)/urdf/workspace_components.xacro"/>
+  <xacro:include filename="$(find godel_robot_config)/urdf/blending_eff_macro.xacro"/>
+  <!-- property list -->
+  <xacro:property name="workcell_height" value="1"/>
+  <xacro:property name="coupler_height" value="0.0"/> <!--"0.087"-->
+  <xacro:property name="arm_prefix" value=""/>
+  <xacro:property name="no_go_height" value="0.1"/>
+  <!-- instantiating workcell definitions -->
+  <xacro:workcell_zone1_components/>
+  <!-- instantiating arm  -->
+  <xacro:abb_irb6640 prefix="${arm_prefix}"/>
+  <!-- instantiating end effector  -->
+  <xacro:blending_eff_definition prefix="${arm_prefix}" eff_adjustment="0.0575"/>
+  <!-- Attach the end effector to the end of the robot arm (tool0) -->
+  <joint name="link_t_to_eff" type="fixed">
+    <parent link="tool0"/>
+    <child link="eff_frame"/>
+    <origin xyz="0 ${coupler_height} 0" rpy="0.0 0.0 3.1416"/>
+  </joint>
+  <!-- start of arm-workcell joint definitions -->
+  <joint name="world_to_base" type="fixed">
+    <parent link="world_frame"/>
+    <child link="${arm_prefix}base_link"/>
+    <origin xyz="0.241 0 0" rpy="0 0 0"/>
+  </joint>
+  <!-- As a work-around for the lack of collision detection with move-it joint
+     moves with the work objects, we use a no-go-zone to prevent the robot
+     from getting too close to the table. Descartes is still unawares, though -->
+  <link name="no_go_zone">
+    <collision>
+      <geometry>
+        <box size="0.8 2.220 ${no_go_height}"/>
+      </geometry>
+    </collision>
+  </link>
+  <joint name="world_to_no_go" type="fixed">
+    <parent link="world_frame" />
+    <child link="no_go_zone" />
+    <origin xyz="1.0 0 ${no_go_height/2.0} " />
+  </joint>
 </robot>

File: godel_robot_config/urdf/sia20d_workspace.xacro (robot description, xacro)
@@ -1,56 +1,44 @@
 <?xml version="1.0" ?>
 <robot name="sia20d_workspace" xmlns:xacro="http://ros.org/wiki/xacro">
-	<xacro:include filename="$(find motoman_sia20d_support)/urdf/sia20d_macro.xacro"/>
-	<xacro:include filename="$(find godel_robot_config)/urdf/workspace_components_swri.xacro"/>
-	<xacro:include filename="$(find godel_robot_config)/urdf/blending_eff_macro.xacro"/>
-	<!-- property list -->
-	<xacro:property name="workcell_height" value="1"/>
-	<xacro:property name="coupler_height" value="0.0"/> <!--"0.087"-->
-    <xacro:property name="attached_object_length" value="0.10"/>
-	<xacro:property name="attached_object_width" value="0.10"/>
-	<xacro:property name="attached_object_height" value="0.025"/>
-	<xacro:property name="arm_prefix" value=""/>
-	<xacro:property name="no_go_height" value="0.1"/>
-	<!-- instantiating workcell definitions -->
-	<xacro:workcell_swri_zone1_components/>
-	<!-- end of workcell definitions -->
-	<link name="roof1">
-		<collision>
-			<geometry>
-				<box size="1.40 2.220 0.04"/>
-			</geometry>
-		</collision>
-	</link>-
-	<link name="no_go_zone">
-		<collision>
-			<geometry>
-				<box size="0.8 2.220 ${no_go_height}"/>
-			</geometry>
-		</collision>
-	</link>
-	<!-- instantiating arm  -->
-	<xacro:blending_eff_definition prefix="${arm_prefix}" eff_adjustment="0.0575"/>
-	<xacro:motoman_sia20d prefix="${arm_prefix}"/>
-	<joint name="link_t_to_eff" type="fixed">
-		<parent link="tool0"/>
-		<child link="eff_frame"/>
-		<origin xyz="0 ${coupler_height} 0" rpy="0.0 0.0 3.1416"/>
-	</joint>
-	<!-- start of arm-workcell joint definitions -->
-	<joint name="world_to_base" type="fixed">
-		<parent link="world_frame"/>
-		<child link="${arm_prefix}base_link"/>
-		<origin xyz="0.241 0 0" rpy="0 0 0"/>
-	</joint>
-	<joint name="world_to_roof1" type="fixed">
-		<parent link="world_frame"/>
-		<child link="roof1"/>
-		<origin xyz="0.65 0 1.32" rpy="0 0 0"/>
-	</joint>
-	<joint name="world_to_no_go" type="fixed">
-		<parent link="world_frame" />
-		<child link="no_go_zone" />
-		<origin xyz="1.0 0 ${no_go_height/2.0} " />
-	</joint>
-	<!-- end of arm-workcell joint definitions -->
+  <xacro:include filename="$(find motoman_sia20d_support)/urdf/sia20d_macro.xacro"/>
+  <xacro:include filename="$(find godel_robot_config)/urdf/workspace_components_swri.xacro"/>
+  <xacro:include filename="$(find godel_robot_config)/urdf/blending_eff_macro.xacro"/>
+  <!-- property list -->
+  <xacro:property name="workcell_height" value="1"/>
+  <xacro:property name="coupler_height" value="0.0"/> <!--"0.087"-->
+  <xacro:property name="arm_prefix" value=""/>
+  <xacro:property name="no_go_height" value="0.1"/>
+  <!-- instantiating workcell definitions -->
+  <xacro:workcell_swri_zone1_components/>
+  <!-- instantiating arm  -->
+  <xacro:motoman_sia20d prefix="${arm_prefix}"/>
+  <!-- instantiating end effector -->
+  <xacro:blending_eff_definition prefix="${arm_prefix}" eff_adjustment="0.0575"/>
+  <!-- Connect tool0 to the end effector -->
+  <joint name="link_t_to_eff" type="fixed">
+    <parent link="tool0"/>
+    <child link="eff_frame"/>
+    <origin xyz="0 ${coupler_height} 0" rpy="0.0 0.0 3.1416"/>
+  </joint>
+  <!-- Connect the world_frame (defined in workcell components) and the robot -->
+  <joint name="world_to_base" type="fixed">
+    <parent link="world_frame"/>
+    <child link="${arm_prefix}base_link"/>
+    <origin xyz="0.241 0 0" rpy="0 0 0"/>
+  </joint>
+  <!-- As a work-around for the lack of collision detection with move-it joint
+       moves with the work objects, we use a no-go-zone to prevent the robot
+       from getting too close to the table. Descartes is still unawares, though -->
+  <link name="no_go_zone">
+    <collision>
+      <geometry>
+        <box size="0.8 2.220 ${no_go_height}"/>
+      </geometry>
+    </collision>
+  </link>
+  <joint name="world_to_no_go" type="fixed">
+    <parent link="world_frame" />
+    <child link="no_go_zone" />
+    <origin xyz="1.0 0 ${no_go_height/2.0} " />
+  </joint>
 </robot>

File: godel_robot_config/urdf/workspace_components.xacro (robot description, xacro)
@@ -84,66 +84,5 @@
 			<origin xyz="${workcell_length * 0.25} 0 0" rpy="0 0 0"/>
 		</joint>
-		<!-- <xacro:workcell_element name="front_wall1" parent="world_frame"
-			 length="0.1" width="2.220" height="${workcell_height}" offset_x="1.3375" offset_y="0"/>
-		<xacro:workcell_element name="back_wall1" parent="world_frame"
-			 length="0.04" width="2.00" height="${workcell_height}" offset_x="0.02" offset_y="0"/>
-		<xacro:workcell_element name="left_wall1" parent="world_frame"
-			 length="1.221" width="0.1" height="${workcell_height}" offset_x="0.687" offset_y="1.060"/>
-		<xacro:workcell_element name="right_wall1" parent="world_frame"
-			 length="1.221" width="0.1" height="${workcell_height}" offset_x="0.687" offset_y="-1.060"/>
-		<xacro:workcell_element name="pole1" parent="world_frame"
-			length="0.09" width="0.09" height="${workcell_height}" offset_x="0.9465" offset_y="-0.845"/> -->
 	</xacro:macro>
 	<!-- end of workcell part1 components macro -->
-	<!-- workcell part2 components macro -->
-	<xacro:macro name="workcell_zone2_components">
-		<link name="table_base2">
-			<visual>
-				<origin xyz="0 0 ${workcell_height * -0.5}" rpy="0 0 0"/>
-				<xacro:workcell_geometry length="${workcell_length * 0.5}"
-					width="${workcell_width}" height="${workcell_height}">
-					<material name="orange_transparent"/>
-				</xacro:workcell_geometry>
-			</visual>
-			<collision>
-				<origin xyz="0 0 ${workcell_height * -0.5}" rpy="0 0 0"/>
-				<xacro:workcell_geometry length="${workcell_length * 0.5}"
-					 width="${workcell_width}" height="${workcell_height}">
-					<material name="blue_transparent"/>
-				</xacro:workcell_geometry>
-			</collision>
-		</link>
-		<link name="roof2">
-			<collision>
-				<origin xyz="0 0 ${workcell_height }" rpy="0 0 0"/>
-				<xacro:workcell_geometry length="${workcell_length * 0.5}"
-					 width="${workcell_width}" height="${workcell_thickness}">
-					<material name="blue_transparent"/>
-				</xacro:workcell_geometry>
-			</collision>
-		</link>
-		<joint name="workcell_to_table_base2" type="fixed">
-			<parent link="world_frame"/>
-			<child link="table_base2"/>
-			<origin xyz="${workcell_length * -0.25} 0 0" rpy="0 0 0"/>
-		</joint>
-		<joint name="workcell_to_roof2" type="fixed">
-			<parent link="world_frame"/>
-			<child link="roof2"/>
-			<origin xyz="${workcell_length * -0.25} 0 0" rpy="0 0 0"/>
-		</joint>
-		<xacro:workcell_element name="front_wall2" parent="world_frame"
-			 length="0.1" width="2.220" height="${workcell_height}" offset_x="-1.3375" offset_y="0"/>
-		<xacro:workcell_element name="back_wall2" parent="world_frame"
-			 length="0.04" width="2.00" height="${workcell_height}" offset_x="0.20" offset_y="0"/>
-		<xacro:workcell_element name="left_wall2" parent="world_frame"
-			length="1.384" width="0.1" height="${workcell_height}" offset_x="-0.601" offset_y="1.060"/>
-		<xacro:workcell_element name="right_wall2" parent="world_frame"
-			length="1.384" width="0.1" height="${workcell_height}" offset_x="-0.601" offset_y="-1.060"/>
-		<xacro:workcell_element name="cover_part1" parent="world_frame"
-			 length="0.229" width="0.508" height="0.14" offset_x="-0.042" offset_y="-0.081"/>
-		<xacro:workcell_element name="cover_part2" parent="world_frame"
-			 length="0.121" width="0.260" height="0.14" offset_x="-0.012" offset_y="-0.465"/>
-	</xacro:macro>
-	<!-- end of workcell part2 components macro -->
 </robot>

File: godel_robot_config/urdf/workspace_components_swri.xacro (robot description, xacro)
@@ -1,4 +1,4 @@
 <?xml version="1.0" ?>
-<robot name="mantis_workspace_components" xmlns:xacro="http://ros.org/wiki/xacro">
+<robot name="swri_workspace_components" xmlns:xacro="http://ros.org/wiki/xacro">
 	<!-- property list -->
 	<xacro:property name="workcell_height" value="1"/>
@@ -79,8 +79,25 @@
 			</collision>
 		</link>
+		<link name="roof1">
+			<collision>
+				<geometry>
+					<box size="1.40 2.220 0.04"/>
+				</geometry>
+			</collision>
+			<visual>
+				<geometry>
+					<box size="1.40 2.220 0.04"/>
+				</geometry>
+			</visual>
+		</link>-
 		<joint name="workcell_to_table_base1" type="fixed">
 			<parent link="world_frame"/>
 			<child link="table_base1"/>
 			<origin xyz="${workcell_length * 0.25} 0 0" rpy="0 0 0"/>
+		</joint>
+		<joint name="workcell_to_roof1" type="fixed">
+			<parent link="world_frame"/>
+			<child link="roof1"/>
+			<origin xyz="0.65 0 1.32" rpy="0 0 0"/>
 		</joint>
 		<xacro:workcell_element name="front_wall1" parent="world_frame"
@@ -96,54 +113,3 @@
 	</xacro:macro>
 	<!-- end of workcell part1 components macro -->
-	<!-- workcell part2 components macro -->
-	<!-- <xacro:macro name="workcell_zone2_components">
-		<link name="table_base2">
-			<visual>
-				<origin xyz="0 0 ${workcell_height * -0.5}" rpy="0 0 0"/>
-				<xacro:workcell_geometry length="${workcell_length * 0.5}"
-					width="${workcell_width}" height="${workcell_height}">
-					<material name="orange_transparent"/>
-				</xacro:workcell_geometry>
-			</visual>
-			<collision>
-				<origin xyz="0 0 ${workcell_height * -0.5}" rpy="0 0 0"/>
-				<xacro:workcell_geometry length="${workcell_length * 0.5}"
-					 width="${workcell_width}" height="${workcell_height}">
-					<material name="blue_transparent"/>
-				</xacro:workcell_geometry>
-			</collision>
-		</link>
-		<link name="roof2">
-			<collision>
-				<origin xyz="0 0 ${workcell_height }" rpy="0 0 0"/>
-				<xacro:workcell_geometry length="${workcell_length * 0.5}"
-					 width="${workcell_width}" height="${workcell_thickness}">
-					<material name="blue_transparent"/>
-				</xacro:workcell_geometry>
-			</collision>
-		</link>
-		<joint name="workcell_to_table_base2" type="fixed">
-			<parent link="world_frame"/>
-			<child link="table_base2"/>
-			<origin xyz="${workcell_length * -0.25} 0 0" rpy="0 0 0"/>
-		</joint>
-		<joint name="workcell_to_roof2" type="fixed">
-			<parent link="world_frame"/>
-			<child link="roof2"/>
-			<origin xyz="${workcell_length * -0.25} 0 0" rpy="0 0 0"/>
-		</joint>
-		<xacro:workcell_element name="front_wall2" parent="world_frame"
-			 length="0.1" width="2.220" height="${workcell_height}" offset_x="-1.3375" offset_y="0"/>
-		<xacro:workcell_element name="back_wall2" parent="world_frame"
-			 length="0.04" width="2.00" height="${workcell_height}" offset_x="0.20" offset_y="0"/>
-		<xacro:workcell_element name="left_wall2" parent="world_frame"
-			length="1.384" width="0.1" height="${workcell_height}" offset_x="-0.601" offset_y="1.060"/>
-		<xacro:workcell_element name="right_wall2" parent="world_frame"
-			length="1.384" width="0.1" height="${workcell_height}" offset_x="-0.601" offset_y="-1.060"/>
-		<xacro:workcell_element name="cover_part1" parent="world_frame"
-			 length="0.229" width="0.508" height="0.14" offset_x="-0.042" offset_y="-0.081"/>
-		<xacro:workcell_element name="cover_part2" parent="world_frame"
-			 length="0.121" width="0.260" height="0.14" offset_x="-0.012" offset_y="-0.465"/>
-	</xacro:macro> -->
-	<!-- end of workcell part2 components macro -->
 </robot>
