Commit message: added asus sensor and all its children links to the final xacro file

File: godel_robot_config/urdf/blending_eff_macro.xacro (robot description, xacro)
@@ -1,61 +1,50 @@
 <?xml version="1.0" ?>
 <robot xmlns:xacro="http://ros.org/wiki/xacro">
+	<xacro:include filename="$(find godel_robot_config)/urdf/asus_sensor_macro.xacro"/>
 	<!-- parameter list -->
 	<xacro:property name="gripper_length" value="0.0"/>
 	<xacro:property name="gripper_width" value="0.0"/>
 	<xacro:property name="gripper_height" value="0.0"/>
-	<xacro:property name="asus_length" value="0.220"/>
-	<xacro:property name="asus_width" value="0.040"/>
-	<xacro:property name="asus_height" value="0.040"/>
-	<xacro:macro name="blending_eff_definition" params="eff_adjustment">
-		<link name="eff_frame"/>
-		<link name="gripper_body">
-			<visual>
-				<geometry>
-					<mesh filename="package://godel_robot_config/meshes/Deburring_eff.STL" />
-				</geometry>
-				<material name="silver">
-					<color rgba="0.8 0.8 0.8 1"/>
-				</material>
-			</visual>
-			<collision>
-				<geometry>
-					<mesh filename="package://godel_robot_config/meshes/Deburring_eff_Collision_Model.STL" />
-				</geometry>
-				<material name="another_blue2">
-					<color rgba="0.38 0.54 0.83 1"/>
-				</material>
-			</collision>
-		</link>
-		<link name="tcp_frame"/>
-		<joint name="gripper_to_palm" type="fixed">
-			<parent link="eff_frame"/>
-			<child link="gripper_body"/>
-			<origin xyz="0 0 ${gripper_height * 0.5}" rpy="0 0 3.6651914"/>
-		</joint>
-		<link name="asus">
-			<visual>
-				<geometry>
-					<box size="${asus_length} ${asus_width} ${asus_height}"/>
-				</geometry>
-				<material name="black"/>
-			</visual>
-			<collision>
-				<geometry>
-					<box size="${asus_length} ${asus_width} ${asus_height}"/>
-				</geometry>
-				<material name="another_blue2"/>
-			</collision>
-		</link>
-		<joint name="eff_frame_to_asus" type="fixed">
-			<parent link="eff_frame"/>
-			<child link="asus"/>
-			<origin xyz="0 0 0.150" rpy="0 0 3.6651914"/>
-		</joint>
-		<joint name="gripper_to_tcp" type="fixed">
-			<parent link="eff_frame"/>
-			<child link="tcp_frame"/>
-			<origin xyz=" 0 ${gripper_length} ${eff_adjustment}" rpy="0 0 0"/>
-		</joint>
+	<xacro:macro name="blending_eff_definition" params="prefix eff_adjustment">
+		<!-- link definition -->
+			<link name="${prefix}eff_frame"/>
+			<link name="${prefix}gripper_body">
+				<visual>
+					<geometry>
+						<mesh filename="package://godel_robot_config/meshes/Deburring_eff.STL" />
+					</geometry>
+					<material name="silver">
+						<color rgba="0.8 0.8 0.8 1"/>
+					</material>
+				</visual>
+				<collision>
+					<geometry>
+						<mesh filename="package://godel_robot_config/meshes/Deburring_eff_Collision_Model.STL" />
+					</geometry>
+					<material name="another_blue2">
+						<color rgba="0.38 0.54 0.83 1"/>
+					</material>
+				</collision>
+			</link>
+			<link name="${prefix}tcp_frame"/>
+			<link name="${prefix}asus_mount"/>
+		<xacro:asus_sensor_definitions prefix="${prefix}" parent_link="${prefix}asus_mount"
+				x_val="0" y_val="0" z_val="0" roll="0.0" pitch="0.0" yaw="0.0"/>
+		<!-- joint definitions -->
+			<joint name="${prefix}gripper_to_palm" type="fixed">
+				<parent link="${prefix}eff_frame"/>
+				<child link="${prefix}gripper_body"/>
+				<origin xyz="0 0 ${gripper_height * 0.5}" rpy="0 0 3.6651914"/>
+			</joint>
+			<joint name="${prefix}eff_frame_to_asus_mount" type="fixed">
+				<parent link="${prefix}eff_frame"/>
+				<child link="${prefix}asus_mount"/>
+				<origin xyz="0 0 0.150" rpy="3.14 0 2.09"/>
+			</joint>
+			<joint name="${prefix}gripper_to_tcp" type="fixed">
+				<parent link="${prefix}eff_frame"/>
+				<child link="${prefix}tcp_frame"/>
+				<origin xyz=" 0 ${gripper_length} ${eff_adjustment}" rpy="0 0 0"/>
+			</joint>
 	</xacro:macro>
 </robot>

File: godel_robot_config/urdf/sia20d_workspace.urdf (robot description, URDF)
Before this commit: robot sia20d_workspace, 24 links, 23 joints
Links:
- added link asus_frame; collision box size=0.04 0.22 0.04; visual box size=0.04 0.22 0.04
- added link asus_ir_link; visual sphere radius=0.0005
- added link asus_ir_optical_frame
- added link asus_link
- added link asus_mount
- added link asus_rgb_link; visual sphere radius=0.0005
- added link asus_rgb_optical_frame
- added link eff_frame
- added link gripper_body; collision mesh filename=package://godel_robot_config/meshes/Deburring_eff_Collision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; visual mesh filename=package://godel_robot_config/meshes/Deburring_eff.STL
- added link tcp_frame
Joints:
- added joint asus_frame_joint: type fixed, parent asus_link, child asus_frame, origin xyz=0 0 0 rpy=0 0 0
- added joint asus_ir_joint: type fixed, parent asus_frame, child asus_ir_link, origin xyz=0 0 0 rpy=0 0 0
- added joint asus_ir_optical_frame_joint: type fixed, parent asus_ir_link, child asus_ir_optical_frame, origin xyz=0 0 0 rpy=-1.57 0 -1.57
- added joint asus_mount_to_asus_link: type fixed, parent asus_mount, child asus_link, origin xyz=0 0 0 rpy=0.0 0.0 0.0
- added joint asus_rgb_joint: type fixed, parent asus_ir_link, child asus_rgb_link, origin xyz=0 -0.03 0 rpy=0 0 0
- added joint asus_rgb_optical_frame_joint: type fixed, parent asus_rgb_link, child asus_rgb_optical_frame, origin xyz=0 0 0 rpy=-1.57 0 -1.57
- added joint eff_frame_to_asus_mount: type fixed, parent eff_frame, child asus_mount, origin xyz=0 0 0.150 rpy=3.14 0 2.09
- added joint gripper_to_palm: type fixed, parent eff_frame, child gripper_body, origin xyz=0 0 0.0 rpy=0 0 3.6651914
- added joint gripper_to_tcp: type fixed, parent eff_frame, child tcp_frame, origin xyz= 0 0.0 0.0 rpy=0 0 0
- added joint link_t_to_eff: type fixed, parent link_t, child eff_frame, origin xyz=0 0.0 0 rpy=0.0 0.0 0.0

File: godel_robot_config/urdf/sia20d_workspace.xacro (robot description, xacro)
@@ -8,5 +8,5 @@
 	<xacro:property name="workcell_height" value="1"/>
 	<xacro:property name="coupler_height" value="0.0"/> <!--"0.087"-->
-        <xacro:property name="attached_object_length" value="0.10"/>
+  <xacro:property name="attached_object_length" value="0.10"/>
 	<xacro:property name="attached_object_width" value="0.10"/>
 	<xacro:property name="attached_object_height" value="0.025"/>
@@ -27,5 +27,5 @@
 	<!-- end of sensor definitions -->
 	<!-- instantiating arm  -->
-	<xacro:blending_eff_definition eff_adjustment="0.0"/>
+	<xacro:blending_eff_definition prefix="${arm_prefix}" eff_adjustment="0.0"/>
 	<xacro:motoman_sia20d prefix="${arm_prefix}"/>
 	<joint name="link_t_to_eff" type="fixed">

Commit message: Adjusted link model and dimensions to put the tool contact point at the correct position. More calibration will be needed

File: godel_robot_config/urdf/blending_eff_macro.xacro (robot description, xacro)
@@ -3,5 +3,5 @@
 	<xacro:include filename="$(find godel_robot_config)/urdf/asus_sensor_macro.xacro"/>
 	<!-- parameter list -->
-	<xacro:property name="gripper_length" value="0.0"/>
+	<xacro:property name="gripper_length" value="0.2"/>
 	<xacro:property name="gripper_width" value="0.0"/>
 	<xacro:property name="gripper_height" value="0.0"/>
@@ -43,7 +43,7 @@
 			</joint>
 			<joint name="${prefix}gripper_to_tcp" type="fixed">
-				<parent link="${prefix}eff_frame"/>
+				<parent link="${prefix}gripper_body"/>
 				<child link="${prefix}tcp_frame"/>
-				<origin xyz=" 0 ${gripper_length} ${eff_adjustment}" rpy="0 0 0"/>
+				<origin xyz="${gripper_length} 0 ${eff_adjustment}" rpy="0 1.57 0"/>
 			</joint>
 	</xacro:macro>

File: godel_robot_config/urdf/sia20d_workspace.xacro (robot description, xacro)
@@ -27,5 +27,5 @@
 	<!-- end of sensor definitions -->
 	<!-- instantiating arm  -->
-	<xacro:blending_eff_definition prefix="${arm_prefix}" eff_adjustment="0.0"/>
+	<xacro:blending_eff_definition prefix="${arm_prefix}" eff_adjustment="0.05"/>
 	<xacro:motoman_sia20d prefix="${arm_prefix}"/>
 	<joint name="link_t_to_eff" type="fixed">

Commit message: Lots of code cleanups.

File: godel_robot_config/urdf/blending_eff_macro.xacro (robot description, xacro)
@@ -45,5 +45,5 @@
 				<parent link="${prefix}gripper_body"/>
 				<child link="${prefix}tcp_frame"/>
-				<origin xyz="${gripper_length} 0 ${eff_adjustment}" rpy="0 1.57 0"/>
+				<origin xyz="${gripper_length} 0 ${eff_adjustment}" rpy="0 1.570796326 0"/>
 			</joint>
 	</xacro:macro>

Commit message: Modified URDF to incorporate laser sensor (very, very roughly)

File: godel_robot_config/urdf/blending_eff_macro.xacro (robot description, xacro)
@@ -2,4 +2,5 @@
 <robot xmlns:xacro="http://ros.org/wiki/xacro">
 	<xacro:include filename="$(find godel_robot_config)/urdf/asus_sensor_macro.xacro"/>
+	<xacro:include filename="$(find keyence_ljv_description)/urdf/lj_v7080_macro.xacro"/>
 	<!-- parameter list -->
 	<xacro:property name="gripper_length" value="0.2"/>
@@ -29,6 +30,9 @@
 			<link name="${prefix}tcp_frame"/>
 			<link name="${prefix}asus_mount"/>
+			<link name="${prefix}keyence_mount"/>
 		<xacro:asus_sensor_definitions prefix="${prefix}" parent_link="${prefix}asus_mount"
 				x_val="0.01479" y_val="0.006741" z_val="0.007162" roll="-3.123031" pitch="0.001618" yaw="0.02739"/>
+		<!-- Keyence sensor -->
+		<xacro:keyence_lj_v7080 prefix="${prefix}keyence_" />
 		<!-- joint definitions -->
 			<joint name="${prefix}gripper_to_palm" type="fixed">
@@ -47,4 +51,14 @@
 				<origin xyz="${gripper_length} 0 ${eff_adjustment}" rpy="0 1.570796326 0"/>
 			</joint>
+			<joint name="${prefix}gripper_to_keyence_mount" type="fixed">
+				<parent link="${prefix}gripper_body" />
+				<child link="${prefix}keyence_mount"/>
+				<origin xyz="-0.15 0 ${gripper_height}" rpy="0 1.57 0" />
+			</joint>
+			<joint name="${prefix}keyence_mount_to_keyence" type="fixed">
+				<parent link="${prefix}keyence_mount"/>
+				<child link="${prefix}keyence_base_link"/>
+				<origin xyz="0 0 0" rpy="0 0 1.57"/>
+			</joint>
 	</xacro:macro>
 </robot>

Commit message: Modified URDF to incorporate laser sensor (very, very roughly)

File: godel_robot_config/urdf/blending_eff_macro.xacro (robot description, xacro)
@@ -2,4 +2,5 @@
 <robot xmlns:xacro="http://ros.org/wiki/xacro">
 	<xacro:include filename="$(find godel_robot_config)/urdf/kinect2_sensor_macro.xacro"/>
+	<xacro:include filename="$(find keyence_ljv_description)/urdf/lj_v7080_macro.xacro"/>
 	<!-- parameter list -->
 	<xacro:property name="gripper_length" value="0.2"/>
@@ -29,6 +30,9 @@
 			<link name="${prefix}tcp_frame"/>
 			<link name="${prefix}kinect2_mount"/>
+			<link name="${prefix}keyence_mount"/>
 		<xacro:kinect2_sensor_definitions prefix="${prefix}" parent_link="${prefix}kinect2_mount"
 				x_val="0.01198326580241401" y_val="-0.06760537682233136" z_val="-0.02237788673513926" roll="-0.008594277487416317" pitch="0.01124423866228241" yaw="0.0007965573534632762"/>
+		<!-- Keyence sensor -->
+		<xacro:keyence_lj_v7080 prefix="${prefix}keyence_" />
 		<!-- joint definitions -->
 			<joint name="${prefix}gripper_to_palm" type="fixed">
@@ -47,4 +51,14 @@
 				<origin xyz="${gripper_length} 0 ${eff_adjustment}" rpy="0 1.570796326 0"/>
 			</joint>
+			<joint name="${prefix}gripper_to_keyence_mount" type="fixed">
+				<parent link="${prefix}gripper_body" />
+				<child link="${prefix}keyence_mount"/>
+				<origin xyz="-0.15 0 ${gripper_height}" rpy="0 1.57 0" />
+			</joint>
+			<joint name="${prefix}keyence_mount_to_keyence" type="fixed">
+				<parent link="${prefix}keyence_mount"/>
+				<child link="${prefix}keyence_base_link"/>
+				<origin xyz="0 0 0" rpy="0 0 1.57"/>
+			</joint>
 	</xacro:macro>
 </robot>

Commit message: Adjusted the model to get the Keyence closer to its actual position

File: godel_robot_config/urdf/blending_eff_macro.xacro (robot description, xacro)
@@ -35,4 +35,10 @@
 		<!-- Keyence sensor -->
 		<xacro:keyence_lj_v7080 prefix="${prefix}keyence_" />
+		<link name="${prefix}keyence_tcp_frame" />
+		<joint name="${prefix}keyence_to_keyence_tcp_frame" type="fixed">
+			<parent link="${prefix}keyence_sensor_optical_frame"/>
+			<child link="${prefix}keyence_tcp_frame"/>
+			<origin rpy="0 3.14159 0"/>
+		</joint>
 		<!-- joint definitions -->
 			<joint name="${prefix}gripper_to_palm" type="fixed">
@@ -54,10 +60,10 @@
 				<parent link="${prefix}gripper_body" />
 				<child link="${prefix}keyence_mount"/>
-				<origin xyz="-0.15 0 ${gripper_height}" rpy="0 1.57 0" />
+				<origin xyz="-0.16 0 0.08" rpy="0 1.570796326 0" />
 			</joint>
 			<joint name="${prefix}keyence_mount_to_keyence" type="fixed">
 				<parent link="${prefix}keyence_mount"/>
 				<child link="${prefix}keyence_base_link"/>
-				<origin xyz="0 0 0" rpy="0 0 1.57"/>
+				<origin xyz="0 0 0" rpy="0 0 1.570796326"/>
 			</joint>
 	</xacro:macro>

Commit message: Updated calibration and added no-go-zone to bottom of the cage

File: godel_robot_config/urdf/blending_eff_macro.xacro (robot description, xacro)
@@ -4,5 +4,5 @@
 	<xacro:include filename="$(find keyence_ljv_description)/urdf/lj_v7080_macro.xacro"/>
 	<!-- parameter list -->
-	<xacro:property name="gripper_length" value="0.2"/>
+	<xacro:property name="gripper_length" value="0.215"/>
 	<xacro:property name="gripper_width" value="0.0"/>
 	<xacro:property name="gripper_height" value="0.0"/>
@@ -32,5 +32,5 @@
 			<link name="${prefix}keyence_mount"/>
 		<xacro:kinect2_sensor_definitions prefix="${prefix}" parent_link="${prefix}kinect2_mount"
-				x_val="0.01198326580241401" y_val="-0.06760537682233136" z_val="-0.02237788673513926" roll="-0.008594277487416317" pitch="0.01124423866228241" yaw="0.0007965573534632762"/>
+				x_val="0.0117323762786166" y_val="-0.05952048473715679" z_val="-0.01945423487488313" roll="-0.006854570337791797" pitch="0.01495538828904983" yaw="0.04379009729706525"/>
 		<!-- Keyence sensor -->
 		<xacro:keyence_lj_v7080 prefix="${prefix}keyence_" />
@@ -39,5 +39,5 @@
 			<parent link="${prefix}keyence_sensor_optical_frame"/>
 			<child link="${prefix}keyence_tcp_frame"/>
-			<origin rpy="0 3.14159 0"/>
+			<origin xyz="0.05 0 0" rpy="0 3.14159 0"/>
 		</joint>
 		<!-- joint definitions -->

File: godel_robot_config/urdf/sia20d_workspace.xacro (robot description, xacro)
@@ -11,4 +11,5 @@
 	<xacro:property name="attached_object_height" value="0.025"/>
 	<xacro:property name="arm_prefix" value=""/>
+	<xacro:property name="no_go_height" value="0.1"/>
 	<!-- instantiating workcell definitions -->
 	<xacro:workcell_zone1_components/>
@@ -18,4 +19,11 @@
 			<geometry>
 				<box size="1.40 2.220 0.04"/>
+			</geometry>
+		</collision>
+	</link>
+	<link name="no_go_zone">
+		<collision>
+			<geometry>
+				<box size="0.8 2.220 ${no_go_height}"/>
 			</geometry>
 		</collision>
@@ -40,4 +48,9 @@
 		<origin xyz="0.65 0 1.32" rpy="0 0 0"/>
 	</joint>
+	<joint name="world_to_no_go" type="fixed">
+		<parent link="world_frame" />
+		<child link="no_go_zone" />
+		<origin xyz="1.0 0 ${no_go_height/2.0} " />
+	</joint>
 	<!-- end of arm-workcell joint definitions -->
 </robot>

Commit message: Updated the surface blending service to add param config windows and the ability to request a save from the GUI

File: godel_robot_config/urdf/blending_eff_macro.xacro (robot description, xacro)
@@ -4,5 +4,5 @@
 	<xacro:include filename="$(find keyence_ljv_description)/urdf/lj_v7080_macro.xacro"/>
 	<!-- parameter list -->
-	<xacro:property name="gripper_length" value="0.215"/>
+	<xacro:property name="gripper_length" value="0.218"/>
 	<xacro:property name="gripper_width" value="0.0"/>
 	<xacro:property name="gripper_height" value="0.0"/>
@@ -32,5 +32,5 @@
 			<link name="${prefix}keyence_mount"/>
 		<xacro:kinect2_sensor_definitions prefix="${prefix}" parent_link="${prefix}kinect2_mount"
-				x_val="0.0117323762786166" y_val="-0.05952048473715679" z_val="-0.01945423487488313" roll="-0.006854570337791797" pitch="0.01495538828904983" yaw="0.04379009729706525"/>
+				x_val="0.01468947476802748" y_val="-0.06367377711162475" z_val="-0.01960868079016488" roll="-0.008749106789621127" pitch="-0.03236299096413636" yaw="0.01705034660528017"/>
 		<!-- Keyence sensor -->
 		<xacro:keyence_lj_v7080 prefix="${prefix}keyence_" />

Commit message: Regenerated the URDFs of all three currently supported robots

File: godel_robot_config/urdf/blending_eff_macro.xacro (robot description, xacro)
@@ -8,27 +8,27 @@
 	<xacro:property name="gripper_height" value="0.0"/>
 	<xacro:macro name="blending_eff_definition" params="prefix eff_adjustment">
-		<!-- link definition -->
-			<link name="${prefix}eff_frame"/>
-			<link name="${prefix}gripper_body">
-				<visual>
-					<geometry>
-						<mesh filename="package://godel_robot_config/meshes/Deburring_eff.STL" />
-					</geometry>
-					<material name="silver">
-						<color rgba="0.8 0.8 0.8 1"/>
-					</material>
-				</visual>
-				<collision>
-					<geometry>
-						<mesh filename="package://godel_robot_config/meshes/Deburring_eff_Collision_Model.STL" />
-					</geometry>
-					<material name="another_blue2">
-						<color rgba="0.38 0.54 0.83 1"/>
-					</material>
-				</collision>
-			</link>
-			<link name="${prefix}tcp_frame"/>
-			<link name="${prefix}kinect2_mount"/>
-			<link name="${prefix}keyence_mount"/>
+			<!-- link definition -->
+		<link name="${prefix}eff_frame"/>
+		<link name="${prefix}gripper_body">
+			<visual>
+				<geometry>
+					<mesh filename="package://godel_robot_config/meshes/Deburring_eff.STL" />
+				</geometry>
+				<material name="silver">
+					<color rgba="0.8 0.8 0.8 1"/>
+				</material>
+			</visual>
+			<collision>
+				<geometry>
+					<mesh filename="package://godel_robot_config/meshes/Deburring_eff_Collision_Model.STL" />
+				</geometry>
+				<material name="another_blue2">
+					<color rgba="0.38 0.54 0.83 1"/>
+				</material>
+			</collision>
+		</link>
+		<link name="${prefix}tcp_frame"/>
+		<link name="${prefix}kinect2_mount"/>
+		<link name="${prefix}keyence_mount"/>
 		<xacro:kinect2_sensor_definitions prefix="${prefix}" parent_link="${prefix}kinect2_mount"
 				x_val="0.01468947476802748" y_val="-0.06367377711162475" z_val="-0.01960868079016488" roll="-0.008749106789621127" pitch="-0.03236299096413636" yaw="0.01705034660528017"/>
@@ -42,29 +42,29 @@
 		</joint>
 		<!-- joint definitions -->
-			<joint name="${prefix}gripper_to_palm" type="fixed">
-				<parent link="${prefix}eff_frame"/>
-				<child link="${prefix}gripper_body"/>
-				<origin xyz="0 0 ${gripper_height * 0.5}" rpy="0 0 3.6651914"/>
-			</joint>
-			<joint name="${prefix}eff_frame_to_kinect2_mount" type="fixed">
-				<parent link="${prefix}eff_frame"/>
-				<child link="${prefix}kinect2_mount"/>
-				<origin xyz="0 0 0.150" rpy="3.14 0 ${2.09+3.141592653589793}"/>
-			</joint>
-			<joint name="${prefix}gripper_to_tcp" type="fixed">
-				<parent link="${prefix}gripper_body"/>
-				<child link="${prefix}tcp_frame"/>
-				<origin xyz="${gripper_length} 0 ${eff_adjustment}" rpy="0 1.570796326 0"/>
-			</joint>
-			<joint name="${prefix}gripper_to_keyence_mount" type="fixed">
-				<parent link="${prefix}gripper_body" />
-				<child link="${prefix}keyence_mount"/>
-				<origin xyz="-0.16 0 0.08" rpy="0 1.570796326 0" />
-			</joint>
-			<joint name="${prefix}keyence_mount_to_keyence" type="fixed">
-				<parent link="${prefix}keyence_mount"/>
-				<child link="${prefix}keyence_base_link"/>
-				<origin xyz="0 0 0" rpy="0 0 1.570796326"/>
-			</joint>
+		<joint name="${prefix}gripper_to_palm" type="fixed">
+			<parent link="${prefix}eff_frame"/>
+			<child link="${prefix}gripper_body"/>
+			<origin xyz="0 0 ${gripper_height * 0.5}" rpy="0 0 3.6651914"/>
+		</joint>
+		<joint name="${prefix}eff_frame_to_kinect2_mount" type="fixed">
+			<parent link="${prefix}eff_frame"/>
+			<child link="${prefix}kinect2_mount"/>
+			<origin xyz="0 0 0.150" rpy="3.14 0 ${2.09+3.141592653589793}"/>
+		</joint>
+		<joint name="${prefix}gripper_to_tcp" type="fixed">
+			<parent link="${prefix}gripper_body"/>
+			<child link="${prefix}tcp_frame"/>
+			<origin xyz="${gripper_length} 0 ${eff_adjustment}" rpy="0 1.570796326 0"/>
+		</joint>
+		<joint name="${prefix}gripper_to_keyence_mount" type="fixed">
+			<parent link="${prefix}gripper_body" />
+			<child link="${prefix}keyence_mount"/>
+			<origin xyz="-0.16 0 0.08" rpy="0 1.570796326 0" />
+		</joint>
+		<joint name="${prefix}keyence_mount_to_keyence" type="fixed">
+			<parent link="${prefix}keyence_mount"/>
+			<child link="${prefix}keyence_base_link"/>
+			<origin xyz="0 0 0" rpy="0 0 1.570796326"/>
+		</joint>
 	</xacro:macro>
 </robot>

Commit message: Updated some planning parameters and succesfuly blended an actual part

File: godel_robot_config/urdf/blending_eff_macro.xacro (robot description, xacro)
@@ -4,5 +4,5 @@
 	<xacro:include filename="$(find keyence_ljv_description)/urdf/lj_v7080_macro.xacro"/>
 	<!-- parameter list -->
-	<xacro:property name="gripper_length" value="0.218"/>
+	<xacro:property name="gripper_length" value="0.195"/>
 	<xacro:property name="gripper_width" value="0.0"/>
 	<xacro:property name="gripper_height" value="0.0"/>
