Commit message: Added Kinect2 camera definitions as well as supporting infastructure for calibrating cameras using the industrial extrinsic cal library!

File: godel_calibration_config/urdf/calib_blending_eff_macro.xacro (robot description, xacro)
@@ -1,10 +1,10 @@
 <?xml version="1.0" ?>
 <robot xmlns:xacro="http://ros.org/wiki/xacro">
-	<xacro:include filename="$(find godel_robot_config)/urdf/kinect2_sensor_macro.xacro"/>
+	<xacro:include filename="$(find godel_calibration_config)/urdf/calib_kinect2_sensor_macro.xacro"/>
 	<!-- parameter list -->
 	<xacro:property name="gripper_length" value="0.2"/>
 	<xacro:property name="gripper_width" value="0.0"/>
 	<xacro:property name="gripper_height" value="0.0"/>
-	<xacro:macro name="blending_eff_definition" params="prefix eff_adjustment">
+	<xacro:macro name="calib_blending_eff_definition" params="prefix eff_adjustment">
 		<!-- link definition -->
 			<link name="${prefix}eff_frame"/>
@@ -29,6 +29,5 @@
 			<link name="${prefix}tcp_frame"/>
 			<link name="${prefix}kinect2_mount"/>
-		<xacro:kinect2_sensor_definitions prefix="${prefix}" parent_link="${prefix}kinect2_mount"
-				x_val="0.01198326580241401" y_val="-0.06760537682233136" z_val="-0.02237788673513926" roll="-0.008594277487416317" pitch="0.01124423866228241" yaw="0.0007965573534632762"/>
+		<xacro:calib_kinect2_sensor_definitions prefix="${prefix}" parent_link="${prefix}kinect2_mount" />
 		<!-- joint definitions -->
 			<joint name="${prefix}gripper_to_palm" type="fixed">

File: godel_robot_config/urdf/sia20d_workspace.urdf (robot description, URDF)
Before this commit: robot sia20d_workspace, 34 links, 33 joints
Links:
- removed link asus_frame
- removed link asus_ir_link
- removed link asus_ir_optical_frame
- removed link asus_link
- removed link asus_mount
- removed link asus_rgb_link
- removed link asus_rgb_optical_frame
- removed link kinect_frame
- removed link kinect_ir_link
- removed link kinect_ir_optical_frame
- removed link kinect_keepout
- removed link kinect_link
- removed link kinect_rgb_link
- removed link kinect_rgb_optical_frame
- added link kinect2_frame; visual box size=0.065 0.25 0.04
- added link kinect2_ir_frame
- added link kinect2_ir_optical_frame
- added link kinect2_link
- added link kinect2_link_pitch
- added link kinect2_link_x_trans; visual sphere radius=0.0005
- added link kinect2_link_y_trans
- added link kinect2_link_yaw
- added link kinect2_link_z_trans
- added link kinect2_mount
- added link kinect2_rgb_frame
- added link kinect2_rgb_optical_frame
- added link target_frame
- added link target_frame_pitch
- added link target_frame_x_trans; visual sphere radius=0.0005
- added link target_frame_y_trans
- added link target_frame_yaw
- added link target_frame_z_trans
Joints:
- removed joint asus_frame_joint
- removed joint asus_ir_joint
- removed joint asus_ir_optical_frame_joint
- removed joint asus_mount_to_asus_link
- removed joint asus_rgb_joint
- removed joint asus_rgb_optical_frame_joint
- removed joint base_link_to_kinect_keepout
- removed joint base_link_to_kinect_link
- removed joint eff_frame_to_asus_mount
- removed joint kinect_frame_joint
- removed joint kinect_ir_joint
- removed joint kinect_ir_optical_frame_joint
- removed joint kinect_rgb_joint
- removed joint kinect_rgb_optical_frame_joint
- added joint eff_frame_to_kinect2_mount: type fixed, parent eff_frame, child kinect2_mount, origin xyz=0 0 0.150 rpy=3.14 0 5.23159265359
- added joint kinect2_frame_joint: type fixed, parent kinect2_link, child kinect2_frame, origin xyz=0 0 0 rpy=0 0 0
- added joint kinect2_ir_joint: type fixed, parent kinect2_frame, child kinect2_ir_frame, origin xyz=0 0.0476 0 rpy=0 0 0
- added joint kinect2_ir_optical_frame_joint: type fixed, parent kinect2_ir_frame, child kinect2_ir_optical_frame, origin xyz=0 0 0 rpy=-1.57 0 -1.57
- added joint kinect2_link_pitch_joint: type revolute, parent kinect2_link_yaw, child kinect2_link_pitch, origin xyz=0 0 0 rpy=0 0 0, axis 0 1 0, limit lower=-3.1415 upper=3.1415 effort=2 velocity=10
- added joint kinect2_link_roll_joint: type revolute, parent kinect2_link_pitch, child kinect2_link, origin xyz=0 0 0 rpy=0 0 0, axis 1 0 0, limit lower=-3.1415 upper=3.1415 effort=2 velocity=10
- added joint kinect2_link_x_joint: type prismatic, parent kinect2_mount, child kinect2_link_x_trans, origin xyz=0 0 0 rpy=0 0 0, axis 1 0 0, limit lower=-1.0 upper=1.0 effort=30 velocity=0.0508
- added joint kinect2_link_y_joint: type prismatic, parent kinect2_link_x_trans, child kinect2_link_y_trans, origin xyz=0 0 0 rpy=0 0 0, axis 0 1 0, limit lower=-1.0 upper=1.0 effort=30 velocity=0.0508
- added joint kinect2_link_yaw_joint: type revolute, parent kinect2_link_z_trans, child kinect2_link_yaw, origin xyz=0 0 0 rpy=0 0 0, axis 0 0 1, limit lower=-3.1415 upper=3.1415 effort=2 velocity=10
- added joint kinect2_link_z_joint: type prismatic, parent kinect2_link_y_trans, child kinect2_link_z_trans, origin xyz=0 0 0 rpy=0 0 0, axis 0 0 1, limit lower=-1.0 upper=1.0 effort=30 velocity=0.0508
- added joint kinect2_rgb_joint: type fixed, parent kinect2_ir_frame, child kinect2_rgb_frame, origin xyz=0 -0.025 0 rpy=0 0 0
- added joint kinect2_rgb_optical_frame_joint: type fixed, parent kinect2_rgb_frame, child kinect2_rgb_optical_frame, origin xyz=0 0 0 rpy=-1.57 0 -1.57
- added joint target_frame_pitch_joint: type revolute, parent target_frame_yaw, child target_frame_pitch, origin xyz=0 0 0 rpy=0 0 0, axis 0 1 0, limit lower=-3.1415 upper=3.1415 effort=2 velocity=10
- added joint target_frame_roll_joint: type revolute, parent target_frame_pitch, child target_frame, origin xyz=0 0 0 rpy=0 0 0, axis 1 0 0, limit lower=-3.1415 upper=3.1415 effort=2 velocity=10
- added joint target_frame_x_joint: type prismatic, parent world_frame, child target_frame_x_trans, origin xyz=0 0 0 rpy=0 0 0, axis 1 0 0, limit lower=-1.0 upper=1.0 effort=30 velocity=0.0508
- added joint target_frame_y_joint: type prismatic, parent target_frame_x_trans, child target_frame_y_trans, origin xyz=0 0 0 rpy=0 0 0, axis 0 1 0, limit lower=-1.0 upper=1.0 effort=30 velocity=0.0508
- added joint target_frame_yaw_joint: type revolute, parent target_frame_z_trans, child target_frame_yaw, origin xyz=0 0 0 rpy=0 0 0, axis 0 0 1, limit lower=-3.1415 upper=3.1415 effort=2 velocity=10
- added joint target_frame_z_joint: type prismatic, parent target_frame_y_trans, child target_frame_z_trans, origin xyz=0 0 0 rpy=0 0 0, axis 0 0 1, limit lower=-1.0 upper=1.0 effort=30 velocity=0.0508
- joint gripper_to_tcp: origin xyz=0.2 0 0.05 rpy=0 0 0 -> xyz=0.2 0 0.05 rpy=0 1.570796326 0
- joint link_t_to_eff: origin xyz=0 0.0 0 rpy=0.0 0.0 0.0 -> xyz=0 0.0 0 rpy=0.0 0.0 3.1416; parent link_t -> tool0

File: godel_robot_config/urdf/sia20d_workspace.xacro (robot description, xacro)
@@ -4,5 +4,4 @@
 	<xacro:include filename="$(find godel_robot_config)/urdf/workspace_components.xacro"/>
 	<xacro:include filename="$(find godel_robot_config)/urdf/blending_eff_macro.xacro"/>
-	<xacro:include filename="$(find godel_robot_config)/urdf/kinect_sensor_macro.xacro"/>
 	<!-- property list -->
 	<xacro:property name="workcell_height" value="1"/>
@@ -22,10 +21,6 @@
 		</collision>
 	</link>
-	<!-- instantiating sensor definitions -->
-	<xacro:sensor_definitions prefix="${arm_prefix}" parent_link="${arm_prefix}base_link"
-		x_val="1.010" y_val="0.169" z_val="1.206" roll="0.005" pitch="1.968" yaw="0.0"/>
-	<!-- end of sensor definitions -->
 	<!-- instantiating arm  -->
-	<xacro:blending_eff_definition prefix="${arm_prefix}" eff_adjustment="0.05"/>
+	<xacro:blending_eff_definition prefix="${arm_prefix}" eff_adjustment="0.0575"/>
 	<xacro:motoman_sia20d prefix="${arm_prefix}"/>
 	<joint name="link_t_to_eff" type="fixed">
