Commit message: add collision model to irb2400 workcell

File: godel_robots/abb/godel_irb2400/godel_irb2400_support/urdf/irb2400_workspace.xacro (robot description, xacro)
@@ -3,4 +3,5 @@
   <xacro:include filename="$(find abb_irb2400_support)/urdf/irb2400_macro.xacro"/>
   <xacro:include filename="$(find blending_end_effector)/urdf/blending_eff_macro.xacro"/>
+  <xacro:include filename="$(find godel_irb2400_support)/urdf/swri_demo_cell_macro.xacro"/>
   <link name="world_frame"/>
   <!-- instantiating arm  -->
@@ -8,4 +9,5 @@
   <!-- instantiating end effector  -->
   <xacro:blending_eff_definition prefix=""/>
+  <xacro:swri_demo_cell prefix=""/>
   <!-- Attach the end effector to the end of the robot arm (tool0) -->
   <joint name="link_t_to_eff" type="fixed">
@@ -20,3 +22,8 @@
     <origin xyz="0 0 0" rpy="0 0 0"/>
   </joint>
+  <joint name="world_to_demo_cell" type="fixed">
+    <parent link="world_frame"/>
+    <child link="demo_cell_base_link"/>
+    <origin xyz="0 0 0" rpy="0 0 0"/>
+  </joint>
 </robot>

Commit message: Recovered the old end effector models from git history. The IRB2400 will continue to use the tool changer. We should really consider breaking out these work spaces.

File: godel_robots/abb/godel_irb2400/godel_irb2400_support/urdf/irb2400_workspace.xacro (robot description, xacro)
@@ -2,6 +2,5 @@
 <robot name="irb2400_workspace" xmlns:xacro="http://ros.org/wiki/xacro">
   <xacro:include filename="$(find abb_irb2400_support)/urdf/irb2400_macro.xacro"/>
-  <xacro:include filename="$(find blending_end_effector)/urdf/blending_eff_macro.xacro"/>
-  <xacro:include filename="$(find godel_irb2400_support)/urdf/swri_demo_cell_macro.xacro"/>
+  <xacro:include filename="$(find godel_irb2400_support)/urdf/abb_blending_eff_macro.xacro"/>
   <link name="world_frame"/>
   <!-- instantiating arm  -->
@@ -9,5 +8,4 @@
   <!-- instantiating end effector  -->
   <xacro:blending_eff_definition prefix=""/>
-  <xacro:swri_demo_cell prefix=""/>
   <!-- Attach the end effector to the end of the robot arm (tool0) -->
   <joint name="link_t_to_eff" type="fixed">
@@ -22,8 +20,3 @@
     <origin xyz="0 0 0" rpy="0 0 0"/>
   </joint>
-  <joint name="world_to_demo_cell" type="fixed">
-    <parent link="world_frame"/>
-    <child link="demo_cell_base_link"/>
-    <origin xyz="0 0 0" rpy="0 0 0"/>
-  </joint>
 </robot>
