Commit message: Added a collision box around the robot.

File: godel_robots/abb/godel_irb1200/godel_irb1200_support/urdf/automate_demo_cell_macro.xacro (robot description, xacro)
@@ -2,12 +2,13 @@
 <!-- Automate 2017 Demo Cell "Structures" -->
 <!-- Exports macro: "xacro:automate_demo_cell" with 1 arg: prefix -->
-<!-- Root link: ${prefix}demo_cell_baselink -->
+<!-- Root link: ${prefix}demo_cell_base_link -->
 <!-- Origin is at the robot (IRB 1200) mounting location -->
 <robot xmlns:xacro="http://ros.org/wiki/xacro">
-  <xacro:property name="demo_cell_width" value="1.778"/> <!--70 in-->
-  <xacro:property name="demo_cell_length" value="1.778"/> <!--70 in-->
-  <xacro:property name="demo_cell_height" value="1.778"/> <!--70 in-->
-  <xacro:property name="robot_to_corner_x" value="-64.668"/> <!-- -25.46 inches -->
-  <xacro:property name="robot_to_corner_y" value="64.668"/> <!-- 25.46 inches -->
+  <xacro:property name="demo_cell_width" value="1.778"/> <!-- Y = 70 in-->
+  <xacro:property name="demo_cell_length" value="1.778"/> <!--X = 70 in-->
+  <xacro:property name="demo_cell_height" value="1.778"/> <!--Z = 70 in-->
+  <xacro:property name="robot_to_corner_x" value="-0.64668"/> <!-- -25.46 inches -->
+  <xacro:property name="robot_to_corner_y" value="-0.64668"/> <!-- -25.46 inches -->
+  <xacro:property name="demo_cell_wall_thickness" value="0.05"/>
   <!--
     The demo cell macro
@@ -16,14 +17,84 @@
   -->
   <xacro:macro name="automate_demo_cell" params="prefix">
-  <link name="${prefix}demo_cell_baselink"/>
+  <link name="${prefix}demo_cell_base_link"/>
   <link name="${prefix}demo_cell_corner"/>
-  <link name="${prefix}demo_cell_back_wall"/>
-  <link name="${prefix}demo_cell_right_wall"/>
-  <link name="${prefix}demo_cell_left_wall"/>
+  <link name="${prefix}demo_cell_back_wall">
+    <collision>
+      <geometry>
+        <box size="${demo_cell_wall_thickness} ${demo_cell_length} ${demo_cell_height}"/>
+      </geometry>
+    </collision>
+  </link>
+  <link name="${prefix}demo_cell_right_wall">
+    <collision>
+      <geometry>
+        <box size="${demo_cell_width} ${demo_cell_wall_thickness} ${demo_cell_height}"/>
+      </geometry>
+    </collision>
+  </link>
+  <link name="${prefix}demo_cell_left_wall">
+    <collision>
+      <geometry>
+        <box size="${demo_cell_width} ${demo_cell_wall_thickness} ${demo_cell_height}"/>
+      </geometry>
+    </collision>
+  </link>
   <!-- light curtains -->
-  <link name="${prefix}demo_cell_front_wall"/>
-  <!--
-  <link name="${prefix}demo_cell_roof"/>
-  <link name="${prefix}demo_cell_floor"/>
+  <link name="${prefix}demo_cell_front_wall">
+    <collision>
+      <geometry>
+        <box size="${demo_cell_wall_thickness} ${demo_cell_length} ${demo_cell_height}"/>
+      </geometry>
+    </collision>
+  </link>
+  <link name="${prefix}demo_cell_roof">
+    <collision>
+      <geometry>
+        <box size="${demo_cell_width} ${demo_cell_length} ${demo_cell_wall_thickness}"/>
+      </geometry>
+    </collision>
+  </link>
+  <link name="${prefix}demo_cell_floor">
+    <collision>
+      <geometry>
+        <box size="${demo_cell_width} ${demo_cell_length} ${demo_cell_wall_thickness}"/>
+      </geometry>
+    </collision>
+  </link>
+  <joint name="${prefix}cell_baselink_to_corner" type="fixed">
+    <parent link="${prefix}demo_cell_base_link"/>
+    <child link="${prefix}demo_cell_corner"/>
+    <origin xyz="${robot_to_corner_x} ${robot_to_corner_y} 0"/>
+  </joint>
+  <joint name="${prefix}cell_corner_to_back" type="fixed">
+    <parent link="${prefix}demo_cell_corner"/>
+    <child link="${prefix}demo_cell_back_wall"/>
+    <origin xyz="${-0.5 * demo_cell_wall_thickness} ${demo_cell_length / 2.0} ${demo_cell_height / 2.0}"/>
+  </joint>
+  <joint name="${prefix}cell_corner_to_left" type="fixed">
+    <parent link="${prefix}demo_cell_corner"/>
+    <child link="${prefix}demo_cell_left_wall"/>
+    <origin xyz="${demo_cell_width / 2.0} ${-0.5 * demo_cell_wall_thickness} ${demo_cell_height / 2.0}"/>
+  </joint>
+  <joint name="${prefix}cell_corner_to_front" type="fixed">
+    <parent link="${prefix}demo_cell_corner"/>
+    <child link="${prefix}demo_cell_front_wall"/>
+    <origin xyz="${demo_cell_width + 0.5 * demo_cell_wall_thickness} ${demo_cell_length / 2.0} ${demo_cell_height / 2.0}"/>
+  </joint>
+  <joint name="${prefix}cell_corner_to_right" type="fixed">
+    <parent link="${prefix}demo_cell_corner"/>
+    <child link="${prefix}demo_cell_right_wall"/>
+    <origin xyz="${demo_cell_width / 2.0} ${demo_cell_length + 0.5 * demo_cell_wall_thickness} ${demo_cell_height / 2.0}"/>
+  </joint>
+  <joint name="${prefix}cell_corner_to_roof" type="fixed">
+    <parent link="${prefix}demo_cell_corner"/>
+    <child link="${prefix}demo_cell_roof"/>
+    <origin xyz="${demo_cell_width / 2.0} ${demo_cell_length / 2.0} ${demo_cell_height + 0.5 * demo_cell_wall_thickness}"/>
+  </joint>
+  <joint name="${prefix}cell_corner_to_floor" type="fixed">
+    <parent link="${prefix}demo_cell_corner"/>
+    <child link="${prefix}demo_cell_floor"/>
+    <origin xyz="${demo_cell_width / 2.0} ${demo_cell_length / 2.0} ${-0.5 * demo_cell_wall_thickness}"/>
+  </joint>
   </xacro:macro>
 </robot>

File: godel_robots/abb/godel_irb1200/godel_irb1200_support/urdf/irb1200_workspace.xacro (robot description, xacro)
@@ -3,4 +3,5 @@
   <xacro:include filename="$(find abb_irb1200_support)/urdf/irb1200_5_90_macro.xacro"/>
   <xacro:include filename="$(find godel_irb1200_support)/urdf/abb_blending_eff_macro.xacro"/>
+  <xacro:include filename="$(find godel_irb1200_support)/urdf/automate_demo_cell_macro.xacro"/>
   <link name="world_frame"/>
   <!-- instantiating arm  -->
@@ -8,4 +9,5 @@
   <!-- instantiating end effector  -->
   <xacro:blending_eff_definition prefix=""/>
+  <xacro:automate_demo_cell prefix=""/>
   <!-- Attach the end effector to the end of the robot arm (tool0) -->
   <joint name="link_t_to_eff" type="fixed">
@@ -20,3 +22,8 @@
     <origin xyz="0 0 0" rpy="0 0 0"/>
   </joint>
+  <joint name="world_to_demo_cell" type="fixed">
+    <parent link="world_frame"/>
+    <child link="demo_cell_base_link"/>
+    <origin xyz="0 0 0" rpy="0 0 0"/>
+  </joint>
 </robot>

Commit message: add visual model of automate cell to xacro

File: godel_robots/abb/godel_irb1200/godel_irb1200_support/urdf/automate_demo_cell_macro.xacro (robot description, xacro)
@@ -17,5 +17,11 @@
   -->
   <xacro:macro name="automate_demo_cell" params="prefix">
-  <link name="${prefix}demo_cell_base_link"/>
+  <link name="${prefix}demo_cell_base_link">
+    <visual>
+      <geometry>
+        <mesh filename="package://godel_irb1200_support/meshes/visual/automate_demo_cell_simplified.dae"/>
+      </geometry>
+    </visual>
+  </link>
   <link name="${prefix}demo_cell_corner"/>
   <link name="${prefix}demo_cell_back_wall">

File: godel_robots/abb/godel_irb1200/godel_irb1200_support/urdf/irb1200_workspace.xacro (robot description, xacro)
@@ -25,5 +25,5 @@
     <parent link="world_frame"/>
     <child link="demo_cell_base_link"/>
-    <origin xyz="0 0 0" rpy="0 0 0"/>
+    <origin xyz="-0.705 -0.718 -0.84775" rpy="1.5707 0 1.5707"/>
   </joint>
 </robot>

Commit message: update urdf for automate and seperate end effector package from abb packages.

File: godel_robots/abb/godel_irb1200/godel_irb1200_support/urdf/automate_demo_cell_macro.xacro (robot description, xacro)
@@ -17,5 +17,14 @@
   -->
   <xacro:macro name="automate_demo_cell" params="prefix">
-  <link name="${prefix}demo_cell_base_link"/>
+  <link name="${prefix}demo_cell_base_link">
+    <visual>
+      <geometry>
+        <mesh filename="package://godel_irb1200_support/meshes/visual/automate_demo_cell_simplified.stl"/>
+      </geometry>
+      <material name="grey">
+        <color rgba="0.5 0.5 0.5 1.0"/>
+      </material>
+    </visual>
+  </link>
   <link name="${prefix}demo_cell_corner"/>
   <link name="${prefix}demo_cell_back_wall">

File: godel_robots/abb/godel_irb1200/godel_irb1200_support/urdf/irb1200_workspace.xacro (robot description, xacro)
@@ -2,5 +2,5 @@
 <robot name="irb1200_workspace" xmlns:xacro="http://ros.org/wiki/xacro">
   <xacro:include filename="$(find abb_irb1200_support)/urdf/irb1200_5_90_macro.xacro"/>
-  <xacro:include filename="$(find godel_irb1200_support)/urdf/abb_blending_eff_macro.xacro"/>
+  <xacro:include filename="$(find blending_end_effector)/urdf/blending_eff_macro.xacro"/>
   <xacro:include filename="$(find godel_irb1200_support)/urdf/automate_demo_cell_macro.xacro"/>
   <link name="world_frame"/>
@@ -14,5 +14,5 @@
     <parent link="tool0"/>
     <child link="eff_frame"/>
-    <origin xyz="0 0 -0.005" rpy="0 0 0${half_pi + half_pi/2.0}"/>
+    <origin xyz="0 0 0" rpy="0 0 3.1415"/>
   </joint>
   <!-- start of arm-workcell joint definitions -->

File: godel_robots/abb/godel_irb2400/godel_irb2400_support/urdf/irb2400_workspace.xacro (robot description, xacro)
@@ -2,5 +2,5 @@
 <robot name="irb2400_workspace" xmlns:xacro="http://ros.org/wiki/xacro">
   <xacro:include filename="$(find abb_irb2400_support)/urdf/irb2400_macro.xacro"/>
-  <xacro:include filename="$(find godel_irb2400_support)/urdf/abb_blending_eff_macro.xacro"/>
+  <xacro:include filename="$(find blending_end_effector)/urdf/blending_eff_macro.xacro"/>
   <link name="world_frame"/>
   <!-- instantiating arm  -->
