Commit message: Tool has different rotation in ABB land

File: godel_robots/abb/godel_irb1200/godel_irb1200_support/urdf/irb1200_workspace.xacro (robot description, xacro)
@@ -14,5 +14,5 @@
     <parent link="tool0"/>
     <child link="eff_frame"/>
-    <origin xyz="0 0 0" rpy="0 0 ${half_pi}"/>
+    <origin xyz="0 0 -0.005" rpy="0 0 0${half_pi + half_pi/2.0}"/>
   </joint>
   <!-- start of arm-workcell joint definitions -->

Commit message: Rotated cage to match the new work cell configuration.

File: godel_robots/abb/godel_irb1200/godel_irb1200_support/urdf/irb1200_workspace.xacro (robot description, xacro)
@@ -25,5 +25,5 @@
     <parent link="world_frame"/>
     <child link="demo_cell_base_link"/>
-    <origin xyz="0 0 0" rpy="0 0 0"/>
+    <origin xyz="0 0 0" rpy="0 0 -${3.14159 / 2.0}"/>
   </joint>
 </robot>
